File: schematics/schematic.brd (EAGLE design)
At the start: 125 x 93 mm, 55 parts, among them IC1 74HC365, T1 BC547, X5 PN61729-S

Commit message: finished first version of schematic;
Parts:
- added C3, C5: 0.1 uF, rcl:C050-025X075
- added C4: 10uF, rcl:E2,5-6
- moved R19 62.7 mm to (60.8, 91.7), turned to 90 degrees
- moved R17 57.1 mm to (19.6, 50.1), flipped to the top, turned to 0 degrees
- moved DEBUG 55.1 mm to (49.8, 77.2), turned to 0 degrees
- moved CLOCK_IN 21.4 mm to (124.6, 97.2)
- moved C2 20.8 mm to (107.1, 49.4), turned to 180 degrees
- moved C1 20.8 mm to (102.5, 19.9)
- moved R23 20.1 mm to (130.1, 34.1)
- moved R5 19.9 mm to (32.0, 81.1), flipped to the top
- moved R22 17.7 mm to (122.4, 34.1)
- moved R20 15.5 mm to (115.1, 90.7), turned to 90 degrees
- moved R27 15.0 mm to (102.0, 44.2), turned to 180 degrees
- moved R26 14.9 mm to (31.0, 89.6), turned to 270 degrees
- moved R1 14.3 mm to (34.5, 34.0), turned to 270 degrees
- moved D1 14.0 mm to (79.7, 91.4), turned to 270 degrees
- moved R4 13.8 mm to (126.3, 34.1)
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Connections:
- removed net GND1: STM32F103.P$21
- net +3V3: now also C5.2
- net +5V: now also C3.1, C4.+
- net GND: now also C3.2, C4.-, C5.1, STM32F103.P$21, STM32F103.P$22
- net PA4: now also LCD.11; no longer LCD.13
- net PA5: now also LCD.12; no longer LCD.14
- net PB10: now also LCD.13; no longer LCD.12
- net PB11: now also LCD.14; no longer LCD.11
Routing:
- net PA6: track 0.00 -> 285.3 mm
- net +5V: track 115.3 -> 304.9 mm, vias 1 -> 0
- net PA1: track 11.8 -> 174.0 mm, vias 0 -> 1
- net PB4: track 0.00 -> 137.3 mm
- net PB1: track 0.00 -> 133.4 mm, vias 0 -> 2
- net PA0: track 7.87 -> 138.8 mm, vias 0 -> 2
- net PB13: track 0.00 -> 118.9 mm
- net PA4: track 0.00 -> 111.1 mm, vias 0 -> 1
- net PA9: track 8.51 -> 116.8 mm, vias 0 -> 2
- net PA5: track 0.00 -> 107.7 mm, vias 0 -> 1
- net PB0: track 33.0 -> 123.8 mm, vias 0 -> 2
- net PB12: track 0.00 -> 90.1 mm
- net PB5: track 0.00 -> 88.8 mm
- net PA2: track 8.16 -> 84.8 mm, vias 0 -> 1
- net N$17: track 0.00 -> 69.9 mm, vias 0 -> 2
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Other:
- board size 125 x 93 mm -> 140 x 100 mm

Commit message: fixed circuit errors
Parts:
- moved R28 1.00 mm to (103.2, 23.2)
Routing:
- net GND: track 666.3 -> 664.4 mm, vias 1 -> 0
Changed lines of the file:
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@@
 <layer number="42" name="bRestrict" color="1" fill="10" visible="yes" active="yes"/>
 <layer number="43" name="vRestrict" color="2" fill="10" visible="yes" active="yes"/>
-<layer number="44" name="Drills" color="7" fill="1" visible="no" active="yes"/>
-<layer number="45" name="Holes" color="7" fill="1" visible="no" active="yes"/>
+<layer number="44" name="Drills" color="7" fill="1" visible="yes" active="yes"/>
+<layer number="45" name="Holes" color="7" fill="1" visible="yes" active="yes"/>
 <layer number="46" name="Milling" color="3" fill="1" visible="no" active="yes"/>
 <layer number="47" name="Measures" color="7" fill="1" visible="no" active="yes"/>
@@
 </layers>
 <board>
+<fusionsync huburn="a.cGVyc29uYWw6dWUyOTRlZjhj" projecturn="a.cGVyc29uYWw6dWUyOTRlZjhjIzIwMTkwMTA1MTY4NDA4MjU2" f3durn="urn:adsk.wipprod:dm.lineage:Lq9hDvX_Sd6aCeZeqRCZkA" pcbguid="abaad317-76b8-409a-97c7-e120a538e6ae" lastpulledtime="" lastsyncedchangeguid="" latestrevisionid="7825f32e-bdc2-458f-9405-eec37679b984" lastsyncedrevisionid="7825f32e-bdc2-458f-9405-eec37679b984" lastboardhashguid="e4f4e491-0abb-39a3-c2ac-01114c3d0e76" lastpushedtime="2021-11-08T23:55:36Z" linktopcb3d="true"/>
 <plain>
 <wire x1="0" y1="0" x2="140" y2="0" width="0" layer="20"/>
@@
 <wire x1="132" y1="21" x2="132" y2="100" width="0.1524" layer="47"/>
 <wire x1="8" y1="21" x2="132" y2="21" width="0.1524" layer="47"/>
+<hole x="4" y="96" drill="3.4"/>
+<hole x="136" y="96" drill="3.4"/>
+<hole x="136" y="4" drill="3.4"/>
+<hole x="4" y="4" drill="3.4"/>
 </plain>
 <attributes>
@@
 <attribute name="VALUE" x="104.2106" y="44.875" size="1.27" layer="27" ratio="10" rot="R180"/>
 </element>
-<element name="R28" library="rcl" library_urn="urn:adsk.eagle:library:334" package="0207/10" package3d_urn="urn:adsk.eagle:package:23491/2" value="100 Ohm" x="102.25" y="23.24" smashed="yes">
-<attribute name="NAME" x="99.202" y="24.764" size="1.27" layer="25" ratio="10"/>
-<attribute name="POPULARITY" value="81" x="134" y="-119" size="1.778" layer="27" display="off"/>
-<attribute name="SPICEPREFIX" value="R" x="134" y="-119" size="1.778" layer="27" display="off"/>
-<attribute name="VALUE" x="99.9894" y="22.605" size="1.27" layer="27" ratio="10"/>
+<element name="R28" library="rcl" library_urn="urn:adsk.eagle:library:334" package="0207/10" package3d_urn="urn:adsk.eagle:package:23491/2" value="100 Ohm" x="103.25" y="23.24" smashed="yes">
+<attribute name="NAME" x="100.202" y="24.764" size="1.27" layer="25" ratio="10"/>
+<attribute name="POPULARITY" value="81" x="135" y="-119" size="1.778" layer="27" display="off"/>
+<attribute name="SPICEPREFIX" value="R" x="135" y="-119" size="1.778" layer="27" display="off"/>
+<attribute name="VALUE" x="100.9894" y="22.605" size="1.27" layer="27" ratio="10"/>
 </element>
 <element name="R3" library="rcl" library_urn="urn:adsk.eagle:library:334" package="0207/10" package3d_urn="urn:adsk.eagle:package:23491/2" value="27 Ohm" x="118.55" y="34.08" smashed="yes" rot="R270">
@@
 <wire x1="82" y1="54.705" x2="89.17" y2="54.705" width="0.8" layer="16"/>
 <wire x1="10.46" y1="87.46" x2="10.5" y2="87.5" width="0.8" layer="16"/>
-<wire x1="10.5" y1="87.5" x2="10.5" y2="90.5" width="0.8" layer="16"/>
-<wire x1="36.05" y1="95.26" x2="43.67" y2="95.26" width="0.8" layer="16"/>
-<wire x1="41.13" y1="95.26" x2="41.13" y2="87.64" width="0.8" layer="16"/>
-<wire x1="43.67" y1="95.26" x2="44.97" y2="93.96" width="0.8" layer="16"/>
 <wire x1="44.97" y1="93.96" x2="48.82" y2="93.96" width="0.8" layer="16"/>
 <wire x1="48.82" y1="93.96" x2="53.78" y2="89" width="0.8" layer="16"/>
@@
 <wire x1="54.75" y1="39.08" x2="54.75" y2="48.75" width="0.8" layer="16"/>
 <wire x1="54.75" y1="48.75" x2="60" y2="54" width="0.8" layer="16"/>
-<wire x1="54.75" y1="39.08" x2="67.92" y2="39.08" width="0.8" layer="16"/>
-<wire x1="67.92" y1="39.08" x2="68" y2="39" width="0.8" layer="16"/>
-<wire x1="68" y1="39" x2="67.77305" y2="38.77305" width="0.8" layer="16"/>
-<wire x1="67.77305" y1="38.77305" x2="67.43" y2="38.77305" width="0.8" layer="16"/>
-<via x="67.43" y="38.77305" extent="1-16" drill="0.35"/>
 <wire x1="52.5" y1="38.5" x2="52.22695" y2="38.77305" width="0.8" layer="16"/>
 <wire x1="52.22695" y1="38.77305" x2="47.19" y2="38.77305" width="0.8" layer="16"/>
@@
 <wire x1="111.69" y1="31.19305" x2="108.80695" y2="31.19305" width="0.8" layer="16"/>
 <wire x1="108.80695" y1="31.19305" x2="106" y2="34" width="0.8" layer="16"/>
-<wire x1="106" y1="34" x2="99.5" y2="34" width="0.8" layer="16"/>
-<wire x1="99.5" y1="34" x2="97.49695" y2="34" width="0.8" layer="16"/>
+<wire x1="106" y1="34" x2="100.5" y2="34" width="0.8" layer="16"/>
+<wire x1="100.5" y1="34" x2="97.49695" y2="34" width="0.8" layer="16"/>
 <wire x1="97.49695" y1="34" x2="97.19" y2="33.69305" width="0.8" layer="16"/>
-<wire x1="104.56" y1="49.42" x2="104.56" y2="39.06" width="0.8" layer="16"/>
-<wire x1="104.56" y1="39.06" x2="99.5" y2="34" width="0.8" layer="16"/>
 <wire x1="109.51" y1="89.24" x2="113.24" y2="89.24" width="0.8" layer="16"/>
 <wire x1="119.055" y1="95.055" x2="124.635" y2="95.055" width="0.8" layer="16"/>
@@
 <wire x1="82" y1="54.705" x2="82" y2="54.63" width="0.4" layer="16"/>
 <wire x1="82" y1="54.63" x2="81.95" y2="54.58" width="0.4" layer="16"/>
-<wire x1="34.31" y1="97" x2="36.05" y2="95.26" width="0.8" layer="16"/>
 <wire x1="24.77" y1="97" x2="34.31" y2="97" width="0.8" layer="16"/>
 <wire x1="49.8" y1="77.15" x2="49.8" y2="85.02" width="0.4" layer="16"/>
@@
 <wire x1="102.185" y1="17.685" x2="102.185" y2="13.685" width="0.8" layer="16"/>
 <wire x1="102.185" y1="13.685" x2="97.64" y2="9.14" width="0.8" layer="16"/>
-<wire x1="41.13" y1="95.26" x2="38.59" y2="95.26" width="0" layer="19" extent="1-1"/>
-<wire x1="36.05" y1="95.26" x2="38.59" y2="95.26" width="0" layer="19" extent="1-1"/>
-<wire x1="10.46" y1="90.17" x2="10.5" y2="90.5" width="0" layer="19" extent="16-16"/>
+<wire x1="34.31" y1="97" x2="36.05" y2="95.26" width="0.8" layer="16"/>
+<wire x1="36.05" y1="95.26" x2="38.59" y2="95.26" width="0.8" layer="16"/>
+<wire x1="38.59" y1="95.26" x2="41.13" y2="95.26" width="0.8" layer="16"/>
+<wire x1="41.13" y1="95.26" x2="43.67" y2="95.26" width="0.8" layer="16"/>
+<wire x1="43.67" y1="95.26" x2="44.97" y2="93.96" width="0.8" layer="16"/>
+<wire x1="41.13" y1="87.64" x2="41.13" y2="95.26" width="0.8" layer="16"/>
+<wire x1="10.5" y1="90.13" x2="10.46" y2="90.17" width="0.8" layer="16"/>
+<wire x1="10.5" y1="87.5" x2="10.5" y2="90.13" width="0.8" layer="16"/>
+<wire x1="54.75" y1="39.08" x2="67.12305" y2="39.08" width="0.8" layer="16"/>
+<wire x1="67.12305" y1="39.08" x2="67.43" y2="38.77305" width="0.8" layer="16"/>
+<wire x1="104.56" y1="49.42" x2="100.5" y2="45.36" width="0.8" layer="16"/>
+<wire x1="100.5" y1="45.36" x2="100.5" y2="34" width="0.8" layer="16"/>
 </signal>
 <signal name="PB12">
@@
 <via x="52.5" y="42.5" extent="1-16" drill="0.35"/>
 <wire x1="61.08" y1="36.23305" x2="54.81305" y2="42.5" width="0.4" layer="1"/>
-<wire x1="54.81305" y1="42.5" x2="52.5" y2="42.5" width="0.4" layer="1"/>
+<wire x1="52.5" y1="42.5" x2="54.81305" y2="42.5" width="0.4" layer="1"/>
 </signal>
 <signal name="N$4">
@@
 <wire x1="14.5" y1="33" x2="20" y2="27.5" width="0.4" layer="1"/>
 <wire x1="20" y1="27.5" x2="28.5" y2="27.5" width="0.4" layer="1"/>
-<wire x1="28.5" y1="27.5" x2="30.5" y2="25.5" width="0.4" layer="1"/>
-<wire x1="30.5" y1="25.5" x2="30.5" y2="20" width="0.4" layer="1"/>
 <wire x1="32.1" y1="69.1" x2="30.5" y2="67.5" width="0.4" layer="1"/>
 <wire x1="30.5" y1="67.5" x2="10.5" y2="67.5" width="0.4" layer="1"/>
 <wire x1="4.5" y1="47.5" x2="14.5" y2="37.5" width="0.4" layer="1"/>
-<wire x1="30.5" y1="20" x2="30.58" y2="20.51" width="0" layer="19" extent="1-1"/>
+<wire x1="30.58" y1="25.42" x2="30.58" y2="20.51" width="0.4" layer="1"/>
+<wire x1="28.5" y1="27.5" x2="30.58" y2="25.42" width="0.4" layer="1"/>
 </signal>
 <signal name="PB4">
@@
 <wire x1="24.73" y1="47.08" x2="27.02" y2="49.37" width="0.4" layer="16"/>
 <wire x1="27.02" y1="49.37" x2="27.02" y2="54.705" width="0.4" layer="16"/>
-<wire x1="105.03" y1="19.92" x2="107.33" y2="22.22" width="0.4" layer="16"/>
-<wire x1="107.33" y1="22.22" x2="107.33" y2="23.24" width="0.4" layer="16"/>
+<wire x1="105.03" y1="19.92" x2="108.33" y2="23.22" width="0.4" layer="16"/>
+<wire x1="108.33" y1="23.22" x2="108.33" y2="23.24" width="0.4" layer="16"/>
 <wire x1="24.73" y1="47.08" x2="24.73" y2="45.73" width="0.4" layer="16"/>
 <wire x1="24.73" y1="45.73" x2="23.5" y2="44.5" width="0.4" layer="16"/>
@@
 <contactref element="ENC" pad="B"/>
 <contactref element="R28" pad="1"/>
-<wire x1="97.19" y1="31.19305" x2="97.19" y2="23.26" width="0.4" layer="16"/>
-<wire x1="97.19" y1="23.26" x2="97.17" y2="23.24" width="0.4" layer="16"/>
+<wire x1="97.19" y1="31.19305" x2="97.19" y2="24.22" width="0.4" layer="16"/>
+<wire x1="97.19" y1="24.22" x2="98.17" y2="23.24" width="0.4" layer="16"/>
 </signal>
 </signals>
@@
 <mfgpreviewcolor name="substratecolor" color="0xFF786E46"/>
 </mfgpreviewcolors>
+<errors>
+</errors>
 </board>
 </drawing>
@@
 </note>
 <note version="8.3" severity="warning">
+Since Version 8.3, EAGLE supports Fusion synchronisation.
+This feature will not be available in this version and saving
+the document will break the link to the Fusion PCB feature.
+</note>
+<note version="8.3" severity="warning">

Commit message: fixed some schematic errors
Connections:
- net GND: no longer X5.S1, X5.S2
Routing:
- net GND: track 664.4 -> 659.1 mm
Changed lines of the file:
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@@
 </layers>
 <board>
-<fusionsync huburn="a.cGVyc29uYWw6dWUyOTRlZjhj" projecturn="a.cGVyc29uYWw6dWUyOTRlZjhjIzIwMTkwMTA1MTY4NDA4MjU2" f3durn="urn:adsk.wipprod:dm.lineage:Lq9hDvX_Sd6aCeZeqRCZkA" pcbguid="abaad317-76b8-409a-97c7-e120a538e6ae" lastpulledtime="" lastsyncedchangeguid="" latestrevisionid="7825f32e-bdc2-458f-9405-eec37679b984" lastsyncedrevisionid="7825f32e-bdc2-458f-9405-eec37679b984" lastboardhashguid="e4f4e491-0abb-39a3-c2ac-01114c3d0e76" lastpushedtime="2021-11-08T23:55:36Z" linktopcb3d="true"/>
+<fusionsync huburn="a.cGVyc29uYWw6dWUyOTRlZjhj" projecturn="a.cGVyc29uYWw6dWUyOTRlZjhjIzIwMTkwMTA1MTY4NDA4MjU2" f3durn="urn:adsk.wipprod:dm.lineage:Lq9hDvX_Sd6aCeZeqRCZkA" pcbguid="" lastpulledtime="" lastsyncedchangeguid="" latestrevisionid="7825f32e-bdc2-458f-9405-eec37679b984" lastsyncedrevisionid="7825f32e-bdc2-458f-9405-eec37679b984" lastboardhashguid="e4f4e491-0abb-39a3-c2ac-01114c3d0e76" lastpushedtime="2021-11-08T23:55:36Z" linktopcb3d="true"/>
 <plain>
 <wire x1="0" y1="0" x2="140" y2="0" width="0" layer="20"/>
@@
 <contactref element="R4" pad="1"/>
 <contactref element="X5" pad="4"/>
-<contactref element="X5" pad="S1"/>
-<contactref element="X5" pad="S2"/>
 <contactref element="M_OUT1" pad="P2"/>
 <contactref element="M_OUT2" pad="P2"/>
@@
 <wire x1="82" y1="54.705" x2="82" y2="54.63" width="0.4" layer="16"/>
 <wire x1="82" y1="54.63" x2="81.95" y2="54.58" width="0.4" layer="16"/>
-<wire x1="24.77" y1="97" x2="34.31" y2="97" width="0.8" layer="16"/>
+<wire x1="24.77" y1="97" x2="25" y2="97" width="0.8" layer="16"/>
+<wire x1="25" y1="97" x2="34.31" y2="97" width="0.8" layer="16"/>
 <wire x1="49.8" y1="77.15" x2="49.8" y2="85.02" width="0.4" layer="16"/>
 <wire x1="49.8" y1="85.02" x2="53.78" y2="89" width="0.4" layer="16"/>
 <wire x1="15.23" y1="87.46" x2="15.23" y2="88.46" width="0.8" layer="16"/>
-<wire x1="16.385" y1="89.615" x2="15.23" y2="88.46" width="0.8" layer="16"/>
-<wire x1="16.385" y1="89.615" x2="21.945" y2="89.615" width="0.8" layer="16"/>
-<wire x1="21.945" y1="89.615" x2="22.5" y2="90.17" width="0.8" layer="16"/>
-<wire x1="22.5" y1="90.17" x2="22.5" y2="94.73" width="0.8" layer="16"/>
-<wire x1="22.5" y1="94.73" x2="24.77" y2="97" width="0.8" layer="16"/>
+<wire x1="16.385" y1="89.615" x2="16.135" y2="89.365" width="0.8" layer="16"/>
+<wire x1="16.135" y1="89.365" x2="15.23" y2="88.46" width="0.8" layer="16"/>
 <wire x1="87.45" y1="42.3" x2="84.91" y2="44.84" width="0.4" layer="16"/>
 <wire x1="84.91" y1="44.84" x2="79.83" y2="44.84" width="0.4" layer="16"/>
@@
 <wire x1="43.67" y1="95.26" x2="44.97" y2="93.96" width="0.8" layer="16"/>
 <wire x1="41.13" y1="87.64" x2="41.13" y2="95.26" width="0.8" layer="16"/>
-<wire x1="10.5" y1="90.13" x2="10.46" y2="90.17" width="0.8" layer="16"/>
-<wire x1="10.5" y1="87.5" x2="10.5" y2="90.13" width="0.8" layer="16"/>
 <wire x1="54.75" y1="39.08" x2="67.12305" y2="39.08" width="0.8" layer="16"/>
 <wire x1="67.12305" y1="39.08" x2="67.43" y2="38.77305" width="0.8" layer="16"/>
 <wire x1="104.56" y1="49.42" x2="100.5" y2="45.36" width="0.8" layer="16"/>
 <wire x1="100.5" y1="45.36" x2="100.5" y2="34" width="0.8" layer="16"/>
+<wire x1="16.385" y1="89.615" x2="23.77" y2="97" width="0.8" layer="16"/>
+<wire x1="23.77" y1="97" x2="24.77" y2="97" width="0.8" layer="16"/>
 </signal>
 <signal name="PB12">
@@
 <contactref element="STM32F103" pad="P$29"/>
 <wire x1="42.26" y1="54.705" x2="42.26" y2="51.24" width="0.4" layer="16"/>
-<wire x1="51" y1="42.5" x2="52.5" y2="42.5" width="0.4" layer="16"/>
-<wire x1="42.26" y1="51.24" x2="51" y2="42.5" width="0.4" layer="16"/>
-<via x="52.5" y="42.5" extent="1-16" drill="0.35"/>
-<wire x1="61.08" y1="36.23305" x2="54.81305" y2="42.5" width="0.4" layer="1"/>
-<wire x1="52.5" y1="42.5" x2="54.81305" y2="42.5" width="0.4" layer="1"/>
+<wire x1="50.5" y1="43" x2="52.5" y2="43" width="0.4" layer="16"/>
+<wire x1="42.26" y1="51.24" x2="50.5" y2="43" width="0.4" layer="16"/>
+<via x="52.5" y="43" extent="1-16" drill="0.35"/>
+<wire x1="61.08" y1="36.23305" x2="54.31305" y2="43" width="0.4" layer="1"/>
+<wire x1="52.5" y1="43" x2="54.31305" y2="43" width="0.4" layer="1"/>
 </signal>
 <signal name="N$4">
